Commit message: Add ur arm to ceiling base robot

File: robots/ceiling_base_arm.urdf.xacro (robot description, xacro)
@@ -1,12 +1,27 @@
 <?xml version="1.0"?>
-<robot name="ceiling" xmlns:xacro="http://wiki.ros.org/xacro">
+<robot name="ceiling_robot" xmlns:xacro="http://wiki.ros.org/xacro">
+	<xacro:arg name="prefix" default="" />
+	<xacro:arg name="hardware_interface" default="PositionJointInterface"/>
 	<xacro:property name="PI" value="3.1415926535897931" />
-	<!-- Import summit XL base elements -->
+    <xacro:property name="arm_position_x" value="0"/>
+    <xacro:property name="arm_position_y" value="0"/>
+    <xacro:property name="arm_position_z" value="0"/>
+    <xacro:property name="arm_orientation_r" value="0"/>
+    <xacro:property name="arm_orientation_p" value="0"/>
+    <xacro:property name="arm_orientation_y" value="0"/>
 	<xacro:include filename="$(find ceiling_arm_description)/urdf/ceiling_base.urdf.xacro" />
+	<xacro:include filename="$(find ur_description)/urdf/inc/ur10_macro.xacro" />
 	<link name="world">
 	</link>
-	<xacro:ceiling_base prefix="test_" parent="world">
+	<xacro:ceiling_base prefix="" parent="world" hardware_interface="$(arg hardware_interface)" >
 		<origin xyz="0.0 0.0 1.0" rpy="0.0 0.0 0.0"/>
 	</xacro:ceiling_base>
+	<xacro:ur10_robot prefix="arm_" transmission_hw_interface="hardware_interface/$(arg hardware_interface)">
+	</xacro:ur10_robot>
+	<joint name="arm_base_joint" type="fixed">
+		<origin xyz="0 0 0" rpy="${PI} 0 0"/>
+		<parent link="connector_link" />
+		<child link="arm_base_link" />
+	</joint>
 	<xacro:ros_control />
 </robot>

File: urdf/ceiling_base.urdf.xacro (robot description, xacro)
@@ -1,11 +1,11 @@
 <?xml version="1.0"?>
-<robot name="ceiling_base_robot" xmlns:xacro="http://wiki.ros.org/xacro">
+<robot name="robot_ceiling_base" xmlns:xacro="http://wiki.ros.org/xacro">
     <xacro:property name="PI" value="3.1415926535897931" />
-    <xacro:macro name="ceiling_base" params="prefix parent *origin">
+    <xacro:macro name="ceiling_base" params="prefix parent hardware_interface:=PositionJointInterface *origin">
         <link name="${prefix}base_long_link">
             <inertial>
-                <mass value="25.0" />
+                <mass value="1.0" />
                 <origin xyz="0 0 0" />
-                <inertia ixx="1.391" ixy="0.004" ixz="0.0" iyy="6.853" iyz="0.0" izz="6.125" />
+                <inertia ixx="1" ixy="0" ixz="0.0" iyy="0.02" iyz="0.0" izz="0.02" />
             </inertial>
             <visual>
@@ -27,7 +27,7 @@
         <link name="${prefix}long_link">
             <inertial>
-                <mass value="25.0" />
+                <mass value="1.0" />
                 <origin xyz="0 0 0" />
-                <inertia ixx="1.391" ixy="0.004" ixz="0.0" iyy="6.853" iyz="0.0" izz="6.125" />
+                <inertia ixx="0.02" ixy="0" ixz="0.0" iyy="0.02" iyz="0.0" izz="0.02" />
             </inertial>
             <visual>
@@ -49,7 +49,7 @@
         <link name="${prefix}base_short_link">
             <inertial>
-                <mass value="25.0" />
+                <mass value="1.0" />
                 <origin xyz="0 0 0" />
-                <inertia ixx="1.391" ixy="0.004" ixz="0.0" iyy="6.853" iyz="0.0" izz="6.125" />
+                <inertia ixx="0.5" ixy="0" ixz="0.0" iyy="0.02" iyz="0.0" izz="0.02" />
             </inertial>
             <visual>
@@ -71,7 +71,7 @@
         <link name="${prefix}short_link">
             <inertial>
-                <mass value="25.0" />
+                <mass value="1.0" />
                 <origin xyz="0 0 0" />
-                <inertia ixx="1.391" ixy="0.004" ixz="0.0" iyy="6.853" iyz="0.0" izz="6.125" />
+                <inertia ixx="0.5" ixy="0" ixz="0.0" iyy="0.02" iyz="0.0" izz="0.02" />
             </inertial>
             <visual>
@@ -95,5 +95,5 @@
                 <mass value="1.0" />
                 <origin xyz="0 0 0" />
-                <inertia ixx="1.391" ixy="0.004" ixz="0.0" iyy="6.853" iyz="0.0" izz="6.125" />
+                <inertia ixx="1e-6" ixy="0" ixz="0.0" iyy="1e-6" iyz="0.0" izz="1e-6" />
             </inertial>
             <visual>
@@ -114,7 +114,5 @@
         </link>
         <joint name="${prefix}base_joint" type="fixed">
-            <!-- TODO add origin from params -->
-            <xacro:insert_block name="origin"/>
-            <!-- <origin rpy="0 0 0" xyz="0 0 0.0" />  -->
+            <xacro:insert_block name="origin" />
             <parent link="${parent}" />
             <child link="${prefix}base_long_link" />
@@ -124,6 +122,7 @@
             <parent link="${prefix}base_long_link" />
             <child link="${prefix}long_link" />
-            <limit effort="30" velocity="1.0" lower="-10" upper="10" />
-            <axis xyz="1 0 0"/>
+            <dynamics damping="1" friction="1"/>
+            <limit effort="300" velocity="5.0" lower="-10" upper="10" />
+            <axis xyz="1 0 0" />
         </joint>
         <joint name="${prefix}base_short_joint" type="fixed">
@@ -136,6 +135,6 @@
             <parent link="${prefix}base_short_link" />
             <child link="${prefix}short_link" />
-            <limit effort="100000.0" velocity="1000.0" lower="0.0" upper="5.0" /> <!-- lower="0.1"
-            upper="0.5" -->
+            <dynamics damping="1" friction="1"/>
+            <limit effort="300" velocity="5.0" lower="0.0" upper="5.0" />
             <axis xyz="0 1 0" />
         </joint>
@@ -145,13 +144,31 @@
             <child link="${prefix}connector_link" />
         </joint>
+        <transmission name="${prefix}long_joint_trans">
+            <type>transmission_interface/SimpleTransmission</type>
+            <joint name="${prefix}long_joint">
+                <hardwareInterface>hardware_interface/${hardware_interface}</hardwareInterface>
+            </joint>
+            <actuator name="${prefix}long_motor">
+                <mechanicalReduction>1</mechanicalReduction>
+            </actuator>
+        </transmission>
+        <transmission name="${prefix}short_joint_trans">
+            <type>transmission_interface/SimpleTransmission</type>
+            <joint name="${prefix}short_joint">
+                <hardwareInterface>hardware_interface/${hardware_interface}</hardwareInterface>
+            </joint>
+            <actuator name="${prefix}short_motor">
+                <mechanicalReduction>1</mechanicalReduction>
+            </actuator>
+        </transmission>
     </xacro:macro>
     <xacro:macro name="ros_control">
         <gazebo>
-          <plugin name="ros_control" filename="libgazebo_ros_control.so">
+            <plugin name="ros_control" filename="libgazebo_ros_control.so">
                 <robotParam>robot_description</robotParam>
-            <controlPeriod>0.001</controlPeriod>
-              <robotSimType>gazebo_ros_control/DefaultRobotHWSim</robotSimType>
+                <controlPeriod>0.001</controlPeriod>
+                <robotSimType>gazebo_ros_control/DefaultRobotHWSim</robotSimType>
                 <legacyModeNS>true</legacyModeNS>
-          </plugin>
+            </plugin>
         </gazebo>
     </xacro:macro>

Commit message: Setup robot

File: robots/ceiling_base_arm.urdf.xacro (robot description, xacro)
@@ -4,18 +4,18 @@
 	<xacro:arg name="hardware_interface" default="PositionJointInterface"/>
 	<xacro:property name="PI" value="3.1415926535897931" />
-    <xacro:property name="arm_position_x" value="0"/>
-    <xacro:property name="arm_position_y" value="0"/>
-    <xacro:property name="arm_position_z" value="0"/>
-    <xacro:property name="arm_orientation_r" value="0"/>
-    <xacro:property name="arm_orientation_p" value="0"/>
-    <xacro:property name="arm_orientation_y" value="0"/>
+    <xacro:property name="robot_position_x" value="0"/>
+    <xacro:property name="robot_position_y" value="0"/>
+    <xacro:property name="robot_position_z" value="0"/>
+    <xacro:property name="robot_orientation_r" value="0"/>
+    <xacro:property name="robot_orientation_p" value="0"/>
+    <xacro:property name="robot_orientation_y" value="0"/>
 	<xacro:include filename="$(find ceiling_arm_description)/urdf/ceiling_base.urdf.xacro" />
 	<xacro:include filename="$(find ur_description)/urdf/inc/ur10_macro.xacro" />
 	<link name="world">
 	</link>
-	<xacro:ceiling_base prefix="" parent="world" hardware_interface="$(arg hardware_interface)" >
-		<origin xyz="0.0 0.0 1.0" rpy="0.0 0.0 0.0"/>
+	<xacro:ceiling_base prefix="$(arg prefix)" parent="world" hardware_interface="$(arg hardware_interface)" >
+		<origin xyz="${robot_position_x} ${robot_position_y} ${robot_position_z}" rpy="${robot_orientation_r} ${robot_orientation_p} ${robot_orientation_y}"/>
 	</xacro:ceiling_base>
-	<xacro:ur10_robot prefix="arm_" transmission_hw_interface="hardware_interface/$(arg hardware_interface)">
+	<xacro:ur10_robot prefix="$(arg prefix)arm_" transmission_hw_interface="hardware_interface/$(arg hardware_interface)">
 	</xacro:ur10_robot>
 	<joint name="arm_base_joint" type="fixed">

File: urdf/ceiling_base.urdf.xacro (robot description, xacro)
@@ -25,4 +25,7 @@
             </collision>
         </link>
+        <!-- <gazebo reference="${prefix}base_long_link">
+            <material>Gazebo/Grey</material>
+        </gazebo> -->
         <link name="${prefix}long_link">
             <inertial>
@@ -54,7 +57,7 @@
             </inertial>
             <visual>
-                <origin xyz="2.4 0 0" rpy="0 0 0" />
+                <origin xyz="1.3 0 0" rpy="0 0 0" />
                 <geometry>
-                    <box size="5.0 0.1 0.01" />
+                    <box size="3.1 0.1 0.01" />
                 </geometry>
                 <material name="Grey">
@@ -63,10 +66,13 @@
             </visual>
             <collision>
-                <origin xyz="2.4 0 0" rpy="0 0 0 " />
+                <origin xyz="1.3 0 0" rpy="0 0 0 " />
                 <geometry>
-                    <box size="5.0 0.1 0.01" />
+                    <box size="3.1 0.1 0.01" />
                 </geometry>
             </collision>
         </link>
+        <!-- <gazebo reference="${prefix}base_short_link">
+            <material>Gazebo/White</material>
+        </gazebo> -->
         <link name="${prefix}short_link">
             <inertial>
@@ -132,5 +138,5 @@
         </joint>
         <joint name="${prefix}short_joint" type="prismatic">
-            <origin rpy="0 0 -${PI/2}" xyz="0 0.0 -0.01" />
+            <origin rpy="0 0 -${PI/2}" xyz="-0.2 0.0 -0.01" />
             <parent link="${prefix}base_short_link" />
             <child link="${prefix}short_link" />
