Commit message: Add hook gripper with arm example

File: robots/ceiling_base.urdf.xacro (robot description, xacro)
@@ -8,5 +8,5 @@
 	</link>
 	<xacro:ceiling_base prefix="$(arg prefix)" parent="world" hardware_interface="$(arg hardware_interface)" >
-		<origin xyz="0.0 0.0 1.0" rpy="0.0 0.0 0.0"/>
+		<origin xyz="0.0 0.0 0.0" rpy="0.0 0.0 0.0"/>
 	</xacro:ceiling_base>
 	<xacro:ros_control />
