Commit message: Add gazebo material color

File: urdf/ceiling_base.urdf.xacro (robot description, xacro)
@@ -25,7 +25,7 @@
             </collision>
         </link>
-        <!-- <gazebo reference="${prefix}base_long_link">
-            <material>Gazebo/Grey</material>
-        </gazebo> -->
+        <gazebo reference="${prefix}base_long_link">
+            <material>Gazebo/Gray</material>
+        </gazebo>
         <link name="${prefix}long_link">
             <inertial>
@@ -72,7 +72,7 @@
             </collision>
         </link>
-        <!-- <gazebo reference="${prefix}base_short_link">
-            <material>Gazebo/White</material>
-        </gazebo> -->
+        <gazebo reference="${prefix}base_short_link">
+            <material>Gazebo/Gray</material>
+        </gazebo>
         <link name="${prefix}short_link">
             <inertial>
